File: Avocado87/Avocado87.kicad_pcb (KiCad board)
At the start: 2 copper layers, 185 parts, among them U1 proton_c

Commit message: Routed PCB
Parts:
- D0, D0A1, D0B1, D0C1, D0D1, D0F1, D0G1, D0H1, D1, D10, D11, D12, D13, D14, D15, D16, D17, D18, D19, D1A1, D1B1, D1C1, D1D1, D1E1, D1F1, D1G1, D1H1, D2, D20, D21, D22, D23, D24, D25, D26, D27, D28, D29, D2A1, D2B1, D2C1, D2D1, D2F1, D2G1, D2H1, D3, D30, D31, D32, D33, D34, D35, D36, D37, D38, D39, D3A1, D3B1, D3C1, D3F1, D3G1, D3H1, D4, D40, D41, D42, D43, D44, D45, D46, D47, D48, D49, D4A1, D4B1, D4C1, D4G1, D5, D50, D51, D52, D58, D59, D5A1, D5F1, D5G1, D5H1, D6, D7, D8, D9: moved to B.Cu
- D55: renamed from D53; moved to B.Cu
- moved D10 319.4 mm to (-130.6, 67.9), turned to 90 degrees
- moved D50 305.9 mm to (-125.6, 140.8), turned to 270 degrees
- moved D20 301.6 mm to (-125.9, 87.0), turned to 90 degrees
- moved D40 296.4 mm to (-118.7, 125.1), turned to 90 degrees
- moved D5H1 292.0 mm to (204.3, 140.8), turned to 270 degrees
- moved D30 289.1 mm to (-123.4, 106.0), turned to 90 degrees
- moved D33 278.0 mm to (-59.2, 106.2), turned to 90 degrees
- moved D3H1 272.3 mm to (204.3, 102.1), turned to 90 degrees
- moved D13 270.1 mm to (-73.4, 67.9), turned to 90 degrees
- moved D2 269.7 mm to (-87.8, 45.0), turned to 90 degrees
- moved D23 260.4 mm to (-63.9, 87.0), turned to 90 degrees
- moved D51 259.3 mm to (-101.7, 140.7), turned to 270 degrees
- moved D2H1 257.8 mm to (204.3, 83.1), turned to 90 degrees
- moved D1H1 253.1 mm to (204.3, 64.0), turned to 90 degrees
- moved D5G1 252.5 mm to (185.3, 140.8), turned to 270 degrees
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Connections:
- D0 pad 1: A9 -> A2
- D0A1 pad 1: A9 -> A2
- D0B1 pad 1: A9 -> A2
- D0C1 pad 1: A9 -> A2
- D0D1 pad 1: A9 -> A2
- D0F1 pad 1: A9 -> A2
- D0G1 pad 1: A9 -> A2
- D0H1 pad 1: A9 -> A2
- D1 pad 1: A9 -> A2
- D10 pad 1: A10 -> B6
- D11 pad 1: A10 -> B6
- D12 pad 1: A10 -> B6
- D13 pad 1: A10 -> B6
- D14 pad 1: A10 -> B6
- D15 pad 1: A10 -> B6
- D16 pad 1: A10 -> B6
- D17 pad 1: A10 -> B6
- D18 pad 1: A10 -> B6
- D19 pad 1: A10 -> B6
- D1A1 pad 1: A10 -> B6
- D1B1 pad 1: A10 -> B6
- D1C1 pad 1: A10 -> B6
- D1D1 pad 1: A10 -> B6
- D1E1 pad 1: A10 -> B6
- D1F1 pad 1: A10 -> B6
- D1G1 pad 1: A10 -> B6
- D1H1 pad 1: A10 -> B6
- D2 pad 1: A9 -> A2
- D20 pad 1: B7 -> B9
- D21 pad 1: B7 -> B9
- D22 pad 1: B7 -> B9
- D23 pad 1: B7 -> B9
- D24 pad 1: B7 -> B9
- D25 pad 1: B7 -> B9
- D26 pad 1: B7 -> B9
- D27 pad 1: B7 -> B9
- D28 pad 1: B7 -> B9
- D29 pad 1: B7 -> B9
- D2A1 pad 1: B7 -> B9
- D2B1 pad 1: B7 -> B9
- D2C1 pad 1: B7 -> B9
- D2D1 pad 1: B7 -> B9
- D2F1 pad 1: B7 -> B9
- D2G1 pad 1: B7 -> B9
- D2H1 pad 1: B7 -> B9
- D3 pad 1: A9 -> A2
- D30 pad 1: B6 -> A15
- D31 pad 1: B6 -> A15
- D32 pad 1: B6 -> A15
- D33 pad 1: B6 -> A15
- D34 pad 1: B6 -> A15
- D35 pad 1: B6 -> A15
- D36 pad 1: B6 -> A15
- D37 pad 1: B6 -> A15
- D38 pad 1: B6 -> A15
- D39 pad 1: B6 -> A15
- D3A1 pad 1: B6 -> A15
- D3B1 pad 1: B6 -> A15
- D3C1 pad 1: B6 -> A15
- D3F1 pad 1: B6 -> A15
- D3G1 pad 1: B6 -> A15
- D3H1 pad 1: B6 -> A15
- D4 pad 1: A9 -> A2
- D40 pad 1: B5 -> A8
- D41 pad 1: B5 -> A8
- D42 pad 1: B5 -> A8
- D43 pad 1: B5 -> A8
- D44 pad 1: B5 -> A8
- D45 pad 1: B5 -> A8
- D46 pad 1: B5 -> A8
- D47 pad 1: B5 -> A8
- D48 pad 1: B5 -> A8
- D49 pad 1: B5 -> A8
- D4A1 pad 1: B5 -> A8
- D4B1 pad 1: B5 -> A8
- D4C1 pad 1: B5 -> A8
- D4G1 pad 1: B5 -> A8
- D5 pad 1: A9 -> A2
- D50 pad 1: B4 -> A7
- D51 pad 1: B4 -> A7
- D52 pad 1: B4 -> A7
- D55 pad 1: B4 -> A7
- D58 pad 1: B4 -> A7
- D59 pad 1: B4 -> A7
- D5A1 pad 1: B4 -> A7
- D5F1 pad 1: B4 -> A7
- D5G1 pad 1: B4 -> A7
- D5H1 pad 1: B4 -> A7
- D6 pad 1: A9 -> A2
- D7 pad 1: A9 -> A2
- D8 pad 1: A9 -> A2
- D9 pad 1: A9 -> A2
- MX0 pad 1: A5 -> B13
- MX0A1 pad 1: B9 -> B2
- MX0B1 pad 1: B15 -> B1
- MX0C1 pad 1: B14 -> A0
- MX0D1 pad 1: B13 -> A1
- MX0F1 pad 1: A0 -> A10
- MX0G1 pad 1: A1 -> A9
- MX0H1 pad 1: A2 -> B7
- MX1 pad 1: A6 -> B14
- MX10 pad 1: A5 -> B13
- MX11 pad 1: A6 -> B14
- MX12 pad 1: A7 -> B15
- MX13 pad 1: A7 -> B10
- MX14 pad 1: A15 -> B11
- MX15 pad 1: A13 -> B12
- MX17 pad 1: B12 -> A13
- MX18 pad 1: B11 -> B4
- MX19 pad 1: B10 -> B3
- MX1A1 pad 1: B9 -> B2
- MX1B1 pad 1: B15 -> B1
- MX1C1 pad 1: B14 -> A0
- MX1D1 pad 1: B13 -> A1
- MX1F1 pad 1: A0 -> A10
- MX1G1 pad 1: A1 -> A9
- MX1H1 pad 1: A2 -> B7
- MX2 pad 1: A7 -> B15
- MX20 pad 1: A5 -> B13
- MX21 pad 1: A6 -> B14
- MX22 pad 1: A7 -> B15
- MX23 pad 1: A7 -> B10
- MX24 pad 1: A15 -> B11
- MX25 pad 1: A13 -> B12
- MX27 pad 1: B12 -> A13
- MX28 pad 1: B11 -> B4
- MX29 pad 1: B10 -> B3
- MX2A1 pad 1: B9 -> B2
- MX2B1 pad 1: B15 -> B1
- MX2C1 pad 1: B14 -> A0
- MX2D1 pad 1: B13 -> A1
- MX2F1 pad 1: A0 -> A10
- MX2G1 pad 1: A1 -> A9
- MX2H1 pad 1: A2 -> B7
- MX3 pad 1: A7 -> B10
- MX30 pad 1: A5 -> B13
- MX31 pad 1: A6 -> B14
- MX32 pad 1: A7 -> B15
- MX33 pad 1: A7 -> B10
- MX34 pad 1: A15 -> B11
- MX35 pad 1: A13 -> B12
- MX37 pad 1: B12 -> A13
- MX38 pad 1: B11 -> B4
- MX39 pad 1: B10 -> B3
- MX3A1 pad 1: B9 -> B2
- MX3B1 pad 1: B15 -> B1
- MX3C1 pad 1: B14 -> A0
- MX3F1 pad 1: A0 -> A10
- MX3G1 pad 1: A1 -> A9
- MX3H1 pad 1: A2 -> B7
- MX4 pad 1: A15 -> B11
- MX40 pad 1: A5 -> B13
- MX41 pad 1: A6 -> B14
- MX42 pad 1: A7 -> B15
- MX43 pad 1: A7 -> B10
- MX44 pad 1: A15 -> B11
- MX45 pad 1: A13 -> B12
- MX47 pad 1: B12 -> A13
- MX48 pad 1: B11 -> B4
- MX49 pad 1: B10 -> B3
- MX4A1 pad 1: B9 -> B2
- MX4B1 pad 1: B15 -> B1
- MX4C1 pad 1: B14 -> A0
- MX4G1 pad 1: A1 -> A9
- MX5 pad 1: A13 -> B12
- MX50 pad 1: A5 -> B13
- MX51 pad 1: A6 -> B14
- MX52 pad 1: A7 -> B15
- MX55 pad 1: A13 -> B12
- MX58 pad 1: B11 -> B4
- MX59 pad 1: B10 -> B3
- MX5A1 pad 1: B9 -> B2
- MX5F1 pad 1: A0 -> A10
- MX5G1 pad 1: A1 -> A9
- MX5H1 pad 1: A2 -> B7
- MX7 pad 1: B12 -> A13
- MX8 pad 1: B11 -> B4
- MX9 pad 1: B10 -> B3
- U1 pad A5: A5 -> (no net)
- U1 pad A6: A6 -> (no net)
- U1 pad A8: A7 -> A8
- U1 pad B1: (no net) -> B1
- U1 pad B2: (no net) -> B2
- U1 pad B3: (no net) -> B3
- U1 pad B5: B5 -> (no net)
Routing:
- net B9: track 0.00 -> 461.2 mm
- net A7: track 0.00 -> 442.2 mm, vias 0 -> 1
- net B6: track 0.00 -> 440.8 mm
- net A15: track 0.00 -> 432.1 mm
- net A8: track 0.00 -> 424.4 mm, vias 0 -> 1
- net A2: track 0.00 -> 424.3 mm
- net B13: track 0.00 -> 399.9 mm
- net B14: track 0.00 -> 396.9 mm
- net B15: track 0.00 -> 377.7 mm
- net B10: track 0.00 -> 310.8 mm
- net B12: track 0.00 -> 303.5 mm
- net B4: track 0.00 -> 298.0 mm
- net B11: track 0.00 -> 293.3 mm
- net B3: track 0.00 -> 286.4 mm
- net B2: track 0.00 -> 268.9 mm
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- added copper zone on F.Cu, net GND
Other:
- board text added: "Avocado87 TKL"
- board text added: "prototype by yanfali (c) 2019"

Commit message: missing line
Routing:
- net A2: track 424.3 -> 444.0 mm

Commit message: Fine tuning
Connections:
- MX0C1 pad 1: A0 -> A1
- MX0D1 pad 1: A1 -> A0
- MX1C1 pad 1: A0 -> A1
- MX1D1 pad 1: A1 -> A0
- MX2C1 pad 1: A0 -> A1
- MX2D1 pad 1: A1 -> A0
- MX3C1 pad 1: A0 -> A1
- MX4C1 pad 1: A0 -> A1
Routing:
- net A0: track 150.8 -> 72.6 mm
- net A1: track 71.6 -> 147.6 mm

Commit message: Fix GND fill
Routing:
- net B7: track 158.7 -> 160.7 mm
Changed lines of the file:
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@@
     (thickness 1.6)
     (drawings 2)
-    (tracks 940)
+    (tracks 944)
     (zones 0)
     (modules 185)
@@
   (segment (start 188.1505 41.783) (end 192.24625 45.87875) (width 0.25) (layer F.Cu) (net 7))
   (segment (start 159.905998 41.783) (end 188.1505 41.783) (width 0.25) (layer F.Cu) (net 7))
-  (segment (start 158.451008 43.23799) (end 159.905998 41.783) (width 0.25) (layer F.Cu) (net 7))
   (segment (start 151.6756 43.23799) (end 158.451008 43.23799) (width 0.25) (layer F.Cu) (net 7))
+  (segment (start 149.098 44.323) (end 149.6695 43.7515) (width 0.25) (layer F.Cu) (net 7))
+  (segment (start 149.098 48.133) (end 149.098 44.323) (width 0.25) (layer F.Cu) (net 7))
+  (segment (start 151.892 49.53) (end 151.257 48.895) (width 0.25) (layer F.Cu) (net 7))
+  (segment (start 158.451008 43.23799) (end 159.905998 41.783) (width 0.25) (layer F.Cu) (net 7))
+  (segment (start 151.892 53.818) (end 151.892 49.53) (width 0.25) (layer F.Cu) (net 7))
+  (segment (start 149.86 48.895) (end 149.098 48.133) (width 0.25) (layer F.Cu) (net 7))
   (segment (start 151.16209 43.7515) (end 151.6756 43.23799) (width 0.25) (layer F.Cu) (net 7))
   (segment (start 149.6695 43.7515) (end 151.16209 43.7515) (width 0.25) (layer F.Cu) (net 7))
-  (segment (start 149.110001 53.870001) (end 149.110001 44.310999) (width 0.25) (layer F.Cu) (net 7))
-  (segment (start 149.110001 44.310999) (end 149.6695 43.7515) (width 0.25) (layer F.Cu) (net 7))
-  (segment (start 150.475 55.235) (end 149.110001 53.870001) (width 0.25) (layer F.Cu) (net 7))
+  (segment (start 151.257 48.895) (end 149.86 48.895) (width 0.25) (layer F.Cu) (net 7))
+  (segment (start 150.475 55.235) (end 151.892 53.818) (width 0.25) (layer F.Cu) (net 7))
   (segment (start -55.373 43.308) (end -55.40375 43.33875) (width 0.25) (layer B.Cu) (net 8))
   (segment (start -49.784 43.308) (end -55.373 43.308) (width 0.25) (layer B.Cu) (net 8))
@@
   (segment (start -142.71625 47.46974) (end -142.621 47.56499) (width 0.25) (layer F.Cu) (net 69))
   (segment (start -142.71625 45.87875) (end -142.71625 47.46974) (width 0.25) (layer F.Cu) (net 69))
+  (segment (start 104.93375 73.66) (end 119.22125 87.9475) (width 0.25) (layer F.Cu) (net 70))
+  (segment (start 104.93375 68.8975) (end 104.93375 73.66) (width 0.25) (layer F.Cu) (net 70))
+  (segment (start 124.333 49.49825) (end 104.93375 68.8975) (width 0.25) (layer F.Cu) (net 70))
+  (segment (start 124.333 46.228) (end 124.333 49.49825) (width 0.25) (layer F.Cu) (net 70))
+  (segment (start 123.98375 45.87875) (end 124.333 46.228) (width 0.25) (layer F.Cu) (net 70))
+  (segment (start 123.98375 45.87875) (end 124.714 46.609) (width 0.25) (layer F.Cu) (net 70))
+  (segment (start 124.333 49.49825) (end 124.333 49.531411) (width 0.25) (layer F.Cu) (net 70))
+  (segment (start 135.245 60.315) (end 135.26 60.315) (width 0.25) (layer F.Cu) (net 70))
+  (segment (start 124.333 49.49825) (end 124.42825 49.49825) (width 0.25) (layer F.Cu) (net 70))
+  (segment (start 124.42825 49.49825) (end 135.245 60.315) (width 0.25) (layer F.Cu) (net 70))
   (segment (start 100.80625 53.975) (end 85.88375 68.8975) (width 0.25) (layer F.Cu) (net 71))
   (segment (start 100.80625 46.51375) (end 100.80625 53.975) (width 0.25) (layer F.Cu) (net 71))
@@
   (segment (start 112.7125 107.6325) (end 112.7125 114.77625) (width 0.25) (layer F.Cu) (net 71))
   (segment (start 112.0775 106.9975) (end 112.7125 107.6325) (width 0.25) (layer F.Cu) (net 71))
-  (segment (start 104.93375 73.66) (end 119.22125 87.9475) (width 0.25) (layer F.Cu) (net 70))
-  (segment (start 104.93375 68.8975) (end 104.93375 73.66) (width 0.25) (layer F.Cu) (net 70))
-  (segment (start 124.333 49.49825) (end 104.93375 68.8975) (width 0.25) (layer F.Cu) (net 70))
-  (segment (start 124.333 46.228) (end 124.333 49.49825) (width 0.25) (layer F.Cu) (net 70))
-  (segment (start 123.98375 45.87875) (end 124.333 46.228) (width 0.25) (layer F.Cu) (net 70))
-  (segment (start 123.98375 45.87875) (end 124.714 46.609) (width 0.25) (layer F.Cu) (net 70))
-  (segment (start 124.333 49.49825) (end 124.333 49.531411) (width 0.25) (layer F.Cu) (net 70))
-  (segment (start 135.245 60.315) (end 135.26 60.315) (width 0.25) (layer F.Cu) (net 70))
-  (segment (start 124.333 49.49825) (end 124.42825 49.49825) (width 0.25) (layer F.Cu) (net 70))
-  (segment (start 124.42825 49.49825) (end 135.245 60.315) (width 0.25) (layer F.Cu) (net 70))
   (segment (start 134.057919 57.775) (end 135.26 57.775) (width 0.25) (layer F.Cu) (net 71))
   (segment (start 100.17125 45.87875) (end 121.63425 45.87875) (width 0.25) (layer F.Cu) (net 71))

Commit message: routing
Routing:
- net B3: track 286.4 -> 285.1 mm
- net B4: track 298.0 -> 297.3 mm
Changed lines of the file:
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@@
     (thickness 1.6)
     (drawings 2)
-    (tracks 944)
+    (tracks 942)
     (zones 0)
     (modules 185)
@@
   (page A4)
   (layers
-    (0 F.Cu signal)
+    (0 F.Cu signal hide)
     (31 B.Cu signal)
     (32 B.Adhes user)
@@
   (segment (start 34.13125 126.6825) (end 34.13125 129.38125) (width 0.25) (layer F.Cu) (net 12))
   (segment (start 33.49625 126.0475) (end 34.13125 126.6825) (width 0.25) (layer F.Cu) (net 12))
-  (segment (start 137.033 72.48982) (end 137.033 90.761002) (width 0.25) (layer B.Cu) (net 12))
+  (segment (start 134.252992 93.54101) (end 37.42774 93.54101) (width 0.25) (layer B.Cu) (net 12))
   (segment (start 37.42774 93.54101) (end 23.97125 106.9975) (width 0.25) (layer B.Cu) (net 12))
+  (segment (start 137.033 72.48982) (end 137.033 90.761002) (width 0.25) (layer B.Cu) (net 12))
+  (segment (start 146.65782 62.865) (end 137.033 72.48982) (width 0.25) (layer B.Cu) (net 12))
   (segment (start 137.033 90.761002) (end 134.252992 93.54101) (width 0.25) (layer B.Cu) (net 12))
-  (segment (start 147.47781 62.04501) (end 137.033 72.48982) (width 0.25) (layer B.Cu) (net 12))
-  (segment (start 148.40501 62.04501) (end 147.47781 62.04501) (width 0.25) (layer B.Cu) (net 12))
-  (segment (start 134.252992 93.54101) (end 37.42774 93.54101) (width 0.25) (layer B.Cu) (net 12))
-  (segment (start 150.475 62.855) (end 149.272919 62.855) (width 0.25) (layer B.Cu) (net 12))
-  (segment (start 148.405081 62.045081) (end 148.40501 62.04501) (width 0.25) (layer B.Cu) (net 12))
-  (segment (start 148.463 62.045081) (end 148.405081 62.045081) (width 0.25) (layer B.Cu) (net 12))
-  (segment (start 149.272919 62.855) (end 148.463 62.045081) (width 0.25) (layer B.Cu) (net 12))
+  (segment (start 148.463 62.865) (end 146.65782 62.865) (width 0.25) (layer B.Cu) (net 12))
+  (segment (start 148.473 62.855) (end 148.463 62.865) (width 0.25) (layer B.Cu) (net 12))
+  (segment (start 150.475 62.855) (end 148.473 62.855) (width 0.25) (layer B.Cu) (net 12))
   (segment (start 6.5395 43.308) (end 6.50875 43.33875) (width 0.25) (layer B.Cu) (net 13))
   (segment (start 12.319 43.308) (end 6.5395 43.308) (width 0.25) (layer B.Cu) (net 13))
@@
   (segment (start 53.18125 126.6825) (end 53.18125 129.38125) (width 0.25) (layer F.Cu) (net 113))
   (segment (start 52.54625 126.0475) (end 53.18125 126.6825) (width 0.25) (layer F.Cu) (net 113))
-  (segment (start 134.439392 93.99102) (end 56.134 93.99102) (width 0.25) (layer B.Cu) (net 113))
-  (segment (start 137.483009 90.947403) (end 134.439392 93.99102) (width 0.25) (layer B.Cu) (net 113))
-  (segment (start 137.48301 72.67622) (end 137.483009 90.947403) (width 0.25) (layer B.Cu) (net 113))
-  (segment (start 146.303475 63.855755) (end 137.48301 72.67622) (width 0.25) (layer B.Cu) (net 113))
-  (segment (start 148.935755 63.855755) (end 146.303475 63.855755) (width 0.25) (layer B.Cu) (net 113))
-  (segment (start 150.475 65.395) (end 148.935755 63.855755) (width 0.25) (layer B.Cu) (net 113))
   (segment (start 38.25875 102.235) (end 39.004875 102.981125) (width 0.25) (layer F.Cu) (net 113))
   (segment (start 38.25875 87.9475) (end 38.25875 102.235) (width 0.25) (layer F.Cu) (net 113))
@@
   (segment (start 38.89375 102.87) (end 39.004875 102.981125) (width 0.25) (layer F.Cu) (net 113))
   (segment (start 43.02125 106.9975) (end 56.02773 93.99102) (width 0.25) (layer B.Cu) (net 113))
+  (segment (start 150.465 65.405) (end 144.75423 65.405) (width 0.25) (layer B.Cu) (net 113))
+  (segment (start 144.75423 65.405) (end 137.48301 72.67622) (width 0.25) (layer B.Cu) (net 113))
+  (segment (start 150.475 65.395) (end 150.465 65.405) (width 0.25) (layer B.Cu) (net 113))
+  (segment (start 137.48301 72.67622) (end 137.483009 90.947403) (width 0.25) (layer B.Cu) (net 113))
+  (segment (start 134.439392 93.99102) (end 56.134 93.99102) (width 0.25) (layer B.Cu) (net 113))
+  (segment (start 137.483009 90.947403) (end 134.439392 93.99102) (width 0.25) (layer B.Cu) (net 113))
   (segment (start 62.70625 53.975) (end 47.78375 68.8975) (width 0.25) (layer F.Cu) (net 114))
   (segment (start 62.70625 46.51375) (end 62.70625 53.975) (width 0.25) (layer F.Cu) (net 114))

Commit message: Add logos for CC NC
Parts:
- added REF**: Symbol_CC-Noncommercial_CopperTop_Small, Symbols:Symbol_CC-Noncommercial_CopperTop_Small, F.Cu at (30.9, 153.0)
- added REF**: Symbol_CC-ShareAlike_CopperTop_Small, Symbols:Symbol_CC-ShareAlike_CopperTop_Small, F.Cu at (24.8, 153.0)
Routing:
- net B6: track 440.8 -> 439.7 mm
- net A7: track 442.2 -> 441.0 mm
- net A15: track 432.1 -> 433.2 mm
Other:
- board text added: "18x6 Matrix using QMK Proton-C"
- board text added: "QMK Powered https://donorbox.org/qmk"
