File: Avocado87/Avocado87.kicad_pcb (KiCad board)
At the start: 2 copper layers, 187 parts, among them U1 proton_c

Commit message: Clean up stuff
Routing:
- net B6: track 128.0 -> 126.0 mm
Changed lines of the file:
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@@
     (thickness 1.6)
     (drawings 11)
-    (tracks 1031)
+    (tracks 1030)
     (zones 0)
     (modules 187)
@@
   (segment (start 156.04198 52.20802) (end 156.15752 52.20802) (width 0.25) (layer B.Cu) (net 9))
   (segment (start 150.475 57.775) (end 156.04198 52.20802) (width 0.25) (layer B.Cu) (net 9))
-  (segment (start 156.15752 52.20802) (end 154.13839 52.20802) (width 0.25) (layer B.Cu) (net 9))
   (segment (start 203.448489 120.615011) (end 203.448489 54.289809) (width 0.25) (layer B.Cu) (net 9))
   (segment (start 200.914 122.9995) (end 201.064 122.9995) (width 0.25) (layer B.Cu) (net 9))
