File: Avocado87/Avocado87.kicad_pcb (KiCad board)
At the start: 2 copper layers, 187 parts, among them U1 proton_c

Commit message: USB pins
Other:
- board text added: "D+"
- board text added: "D-"
- board text added: "Designed in Sunnyvale CA"
- board text added: "Proton-C this Side"
Changed lines of the file:
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@@
   (general
     (thickness 1.6)
-    (drawings 12)
+    (drawings 16)
     (tracks 1030)
     (zones 0)
@@
   (page A4)
   (layers
-    (0 F.Cu signal)
+    (0 F.Cu signal hide)
     (31 B.Cu signal)
     (32 B.Adhes user)
@@
       (net 119 +5V))
   )
-  (gr_text "Avocado87 TKL" (at 154.8765 123.3805) (layer F.SilkS)
+  (gr_text D+ (at 147.955 48.387) (layer B.SilkS)
+    (effects (font (size 1 1) (thickness 0.15)) (justify mirror))
+  )
+  (gr_text D- (at 145.3515 48.4505) (layer B.SilkS)
+    (effects (font (size 1 1) (thickness 0.15)) (justify mirror))
+  )
+  (gr_text "Proton-C this Side" (at 146.7485 62.484 90) (layer B.SilkS)
+    (effects (font (size 1 1) (thickness 0.15)) (justify mirror))
+  )
+  (gr_text "Designed in Sunnyvale CA" (at 154.7495 119.0625) (layer B.SilkS)
+    (effects (font (size 1 1) (thickness 0.15)) (justify mirror))
+  )
+  (gr_text "Avocado87 TKL" (at 154.7495 116.332) (layer B.SilkS)
     (effects (font (size 2 2) (thickness 0.15)) (justify mirror))
   )
